File: src/Electronics/ProtoB/eaglePCB/covid-respirator-ProtoB.brd (EAGLE design)
At the start: 160 x 100 mm, 18 parts, among them IC2 L7805CV-DG, Q1 VNP35N07-E, T2 BC548

Commit message: update protoB schematic
Connections:
- net N$10 renamed A1
- net N$14 renamed D13
- net N$2 renamed D5
- net N$3 renamed A3
- net N$5 renamed D6
- net N$7 renamed AREF
- net N$8 renamed AGND
Changed lines of the file:
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@@
 <contactref element="R1" pad="1"/>
 </signal>
-<signal name="N$2">
+<signal name="D5">
 <contactref element="R1" pad="2"/>
 </signal>
-<signal name="N$3">
+<signal name="A3">
 <contactref element="R2" pad="1"/>
 <contactref element="R3" pad="2"/>
@@
 <wire x1="-49.53" y1="45.72" x2="-21.59" y2="2.54" width="0" layer="19" extent="1-1"/>
 </signal>
-<signal name="N$5">
+<signal name="D6">
 <contactref element="R4" pad="2"/>
 </signal>
-<signal name="N$7">
+<signal name="AREF">
 <contactref element="IC2" pad="3"/>
 <contactref element="C2" pad="+"/>
@@
 <wire x1="-19.05" y1="39.37" x2="-40.3" y2="30.48" width="0" layer="19" extent="1-1"/>
 </signal>
-<signal name="N$8">
+<signal name="AGND">
 <contactref element="C1" pad="-"/>
 <contactref element="C2" pad="-"/>
@@
 <contactref element="R5" pad="2"/>
 </signal>
-<signal name="N$10">
+<signal name="A1">
 <contactref element="R5" pad="1"/>
 <contactref element="C4" pad="1"/>
@@
 <wire x1="-64.77" y1="-20.32" x2="-67.31" y2="-27.94" width="0" layer="19" extent="1-1"/>
 </signal>
-<signal name="N$14">
+<signal name="D13">
 <contactref element="R7" pad="2"/>
 </signal>

Commit message: update power supply and sensors
Parts:
- F1: value 2A -> 8A
Connections:
- removed net N$15: BATTERY.+, F1.1
- new net N$2: BATTERY.-
- new net N$3: BATTERY.+
- new net N$5: F1.1
- net GND: no longer BATTERY.-
Changed lines of the file:
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@@
 <element name="R7" library="rcl" package="0207/10" value="1k" x="-62.23" y="-33.02"/>
 <element name="R8" library="rcl" package="0207/10" value="1k" x="-62.23" y="-38.1"/>
-<element name="F1" library="fuse" package="19560" value="2A" x="-73.66" y="-34.29">
+<element name="F1" library="fuse" package="19560" value="8A" x="-73.66" y="-34.29">
 <attribute name="MPN" value="56000001009" x="-73.66" y="-34.29" size="1.778" layer="27" display="off"/>
 <attribute name="OC_FARNELL" value="1185363" x="-73.66" y="-34.29" size="1.778" layer="27" display="off"/>
@@
 <signals>
 <signal name="GND">
-<contactref element="BATTERY" pad="-"/>
 <contactref element="R3" pad="1"/>
 <contactref element="Q1" pad="3"/>
@@
 <wire x1="-62.23" y1="-20.32" x2="-57.15" y2="-27.94" width="0" layer="19" extent="1-1"/>
 <wire x1="-16.51" y1="2.54" x2="-57.15" y2="-27.94" width="0" layer="19" extent="1-1"/>
-<wire x1="-17.78" y1="27.94" x2="-16.51" y2="2.54" width="0" layer="19" extent="1-1"/>
-<wire x1="-36.83" y1="45.72" x2="-17.78" y2="27.94" width="0" layer="19" extent="1-1"/>
+<wire x1="-36.83" y1="45.72" x2="-16.51" y2="2.54" width="0" layer="19" extent="1-1"/>
 </signal>
 <signal name="+12V">
@@
 <contactref element="R7" pad="2"/>
 </signal>
-<signal name="N$15">
+<signal name="N$2">
+<contactref element="BATTERY" pad="-"/>
+</signal>
+<signal name="N$3">
 <contactref element="BATTERY" pad="+"/>
+</signal>
+<signal name="N$5">
 <contactref element="F1" pad="1"/>
-<wire x1="-17.78" y1="33.02" x2="-76.2" y2="-34.29" width="0" layer="19" extent="1-1"/>
 </signal>
 </signals>
